File: encoder/stator-bot/stator-bot.kicad_pcb (KiCad board)
At the start: 4 copper layers, 75.5 x 36.5 mm, 9 parts, among them U1 STM32G474RBTx, U3 TYPE-C_16PIN_2MD(073), U4 XL-1608SURC-06, U5 AZ1117-3.3

Commit message: xxx
Parts:
- moved C1 34.7 mm to (75.2, 87.5), turned to -90 degrees
- moved U5 31.5 mm to (80.0, 90.0), turned to 90 degrees
- moved U3 28.8 mm to (90.3, 91.6), turned to 0 degrees
- moved R2 21.8 mm to (93.0, 87.5), turned to 0 degrees
- moved C2 20.0 mm to (85.5, 86.5), turned to 0 degrees
- moved R3 18.8 mm to (89.2, 86.7), turned to 90 degrees
- moved U4 16.1 mm to (84.5, 83.8), turned to 180 degrees
- moved R1 13.3 mm to (87.8, 83.8), turned to 0 degrees
- moved U1 5.32 mm to (88.2, 75.2), turned to -90 degrees
Other:
- board size 75.5 x 36.5 mm -> 100 x 100 mm

Commit message: aaaa
Parts:
- added REF**: TO-263-2, Package_TO_SOT_SMD:TO-263-2, F.Cu at (134.8, 57.7)
- added REF**: TO-263-2, Package_TO_SOT_SMD:TO-263-2, F.Cu at (147.0, 83.9)
- added REF**: TO-263-2, Package_TO_SOT_SMD:TO-263-2, F.Cu at (122.2, 57.7)
- added REF**: TO-263-2, Package_TO_SOT_SMD:TO-263-2, F.Cu at (134.4, 83.9)
- added REF**: TO-263-2, Package_TO_SOT_SMD:TO-263-2, F.Cu at (147.0, 57.7)
- added REF**: TO-263-2, Package_TO_SOT_SMD:TO-263-2, F.Cu at (122.2, 83.9)
- moved C1 18.5 mm to (56.8, 87.5)
- moved C2 18.5 mm to (67.0, 86.5)
- moved R1 18.5 mm to (69.2, 83.8)
- moved R2 18.5 mm to (74.5, 87.5)
- moved R3 18.5 mm to (70.8, 86.7)
- moved U1 18.5 mm to (69.8, 75.2)
- moved U3 18.5 mm to (71.8, 91.6)
- moved U4 18.5 mm to (66.0, 83.8)
- moved U5 18.5 mm to (61.5, 90.0)
Other:
- board size 100 x 100 mm -> 178 x 127 mm
