File: encoder/stator-top/stator-top.kicad_pcb (KiCad board)
At the start: 4 copper layers, 0 parts

Commit message: aaaa
Parts:
- added C1: 100n, Capacitor_SMD:C_0603_1608Metric, F.Cu at (77.5, 47.0)
- added C2: 100n, Capacitor_SMD:C_0603_1608Metric, F.Cu at (74.2, 47.0)
- added R1: 10Meg, Resistor_SMD:R_0603_1608Metric, F.Cu at (71.6, 55.9)
- added R2: 20, Resistor_SMD:R_0603_1608Metric, F.Cu at (77.2, 45.5)
- added R3: 10Meg, Resistor_SMD:R_0603_1608Metric, F.Cu at (75.8, 49.0)
- added R4: 20, Resistor_SMD:R_0603_1608Metric, F.Cu at (77.2, 43.2)
- added U2: FH34SRJ-6S-0_5SH(50), footprint:FFC-SMD_6P-P0.50_FH34SRJ-6S-0.5SH, F.Cu at (113.2, 43.5)
- added U3: TLV9062IDGKR, footprint:VSSOP-8_L3.0-W3.0-P0.65-LS4.9-BL, F.Cu at (72.1, 51.0)
- added U4: FH34SRJ-6S-0_5SH(50), footprint:FFC-SMD_6P-P0.50_FH34SRJ-6S-0.5SH, F.Cu at (72.5, 43.5)
Routing:
- net +3.3V: track 0.00 -> 47.7 mm, vias 0 -> 3
- net /RX+: track 0.00 -> 19.4 mm, vias 0 -> 2
- net /BIAS: track 0.00 -> 18.8 mm, vias 0 -> 2
- net /RX-: track 0.00 -> 10.9 mm, vias 0 -> 2
- net /GUARD_RX+: track 0.00 -> 9.60 mm, vias 0 -> 4
- net GND: track 0.00 -> 8.34 mm, vias 0 -> 19
- net /E_RX-: track 0.00 -> 7.93 mm
- net /E_RX+: track 0.00 -> 6.00 mm
- net /GUARD_RX-: track 0.00 -> 5.71 mm, vias 0 -> 3
- added copper zone on F.Cu, net /GUARD_RX+
- added copper zone on In1.Cu, net /GUARD_RX+
- added copper zone on F.Cu, net /GUARD_RX-
- added copper zone on In1.Cu, net /GUARD_RX-
- added copper zone on B.Cu, net GND
- added copper zone on F.Cu, net GND
- added copper zone on In1.Cu, net GND
Other:
- board outline added: 50 x 50 mm
