File: encoder/stator-top/stator-top.kicad_sch (KiCad schematic)
At the start: 0 parts

Commit message: aaaa
Parts:
- added C1, C2: 100n, Capacitor_SMD:C_0603_1608Metric, symbol Device:C
- added R1, R3: 10Meg, Resistor_SMD:R_0603_1608Metric, symbol Device:R
- added R2, R4: 20, Resistor_SMD:R_0603_1608Metric, symbol Device:R
- added U2, U4: FH34SRJ-6S-0_5SH(50), footprint:FFC-SMD_6P-P0.50_FH34SRJ-6S-0.5SH, symbol symbol:FH34SRJ-6S-0_5SH(50)
- added U3: TLV9062IDGKR, footprint:VSSOP-8_L3.0-W3.0-P0.65-LS4.9-BL, symbol symbol:TLV9062IDGKR
Connections:
- new net +3.3V: C2.1, U2.1, U3.8 (V+)
- new net BIAS: C1.1, R1.2, R3.2, U4.6
- new net E_RX+: R1.1, U3.3 (IN1+)
- new net E_RX-: R3.1, U3.5 (IN2+)
- new net GND: C1.2, C2.2, U2.6, U3.4 (V-), U4.1, U4.3, U4.5
- new net GUARD_RX+: R2.2
- new net GUARD_RX-: R4.2
- new net PH2: U2.3
- new net PH3: U2.4
- new net PH4: U2.5
- new net RX+: R2.1, U3.1 (OUT1), U3.2 (IN1-), U4.2
- new net RX-: R4.1, U3.6 (IN2-), U3.7 (OUT2), U4.4
- no-connect marks 0 -> 4
